File: xenlight.sch (EAGLE design)
At the start: 33 parts, among them IC1 MEGA16-A, IC14 FT232RL, IC2 74HC573D, IC3 74HC573D, IC4 74HC573D, IC5 74HC573D, IC6 74HC573D, IC7 74HC573D, X1 057-010-1, X2 057-010-1, X3 057-010-1, X4 057-010-1, X5 057-010-1, X6 057-010-1, X7 KUSBVX

Commit message: Second version of board, not for homemade production.
Connections:
- net GND: no longer IC12.I6, IC12.I7, IC12.I8, IC13.I6, IC13.I7, IC13.I8
- net VCC: now also IC12.I6, IC12.I7, IC12.I8, IC13.I6, IC13.I7, IC13.I8
Changed lines of the file:
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@@
 <attribute name="OC_NEWARK" value="unknown"/>
 </part>
+<part name="P+2" library="supply1" deviceset="VCC" device=""/>
 </parts>
 <sheets>
@@
 <instance part="X5" gate="-9" x="177.8" y="7.62"/>
 <instance part="X5" gate="-10" x="177.8" y="5.08"/>
+<instance part="P+2" gate="VCC" x="162.56" y="12.7" rot="R90"/>
 </instances>
 <busses>
@@
 <pinref part="X6" gate="-2" pin="S"/>
 <wire x1="83.82" y1="114.3" x2="88.9" y2="114.3" width="0.1524" layer="91"/>
+</segment>
+<segment>
+<pinref part="IC12" gate="G$1" pin="I6"/>
+<wire x1="175.26" y1="22.86" x2="167.64" y2="22.86" width="0.1524" layer="91"/>
+<wire x1="167.64" y1="22.86" x2="167.64" y2="20.32" width="0.1524" layer="91"/>
+<pinref part="P+2" gate="VCC" pin="VCC"/>
+<wire x1="167.64" y1="20.32" x2="167.64" y2="17.78" width="0.1524" layer="91"/>
+<wire x1="167.64" y1="17.78" x2="167.64" y2="12.7" width="0.1524" layer="91"/>
+<wire x1="167.64" y1="12.7" x2="165.1" y2="12.7" width="0.1524" layer="91"/>
+<pinref part="IC12" gate="G$1" pin="I7"/>
+<wire x1="175.26" y1="20.32" x2="167.64" y2="20.32" width="0.1524" layer="91"/>
+<pinref part="IC12" gate="G$1" pin="I8"/>
+<wire x1="175.26" y1="17.78" x2="167.64" y2="17.78" width="0.1524" layer="91"/>
+<pinref part="IC13" gate="G$1" pin="I6"/>
+<wire x1="175.26" y1="-12.7" x2="167.64" y2="-12.7" width="0.1524" layer="91"/>
+<wire x1="167.64" y1="-12.7" x2="167.64" y2="12.7" width="0.1524" layer="91"/>
+<pinref part="IC13" gate="G$1" pin="I7"/>
+<wire x1="175.26" y1="-15.24" x2="167.64" y2="-15.24" width="0.1524" layer="91"/>
+<wire x1="167.64" y1="-15.24" x2="167.64" y2="-12.7" width="0.1524" layer="91"/>
+<pinref part="IC13" gate="G$1" pin="I8"/>
+<wire x1="175.26" y1="-17.78" x2="167.64" y2="-17.78" width="0.1524" layer="91"/>
+<wire x1="167.64" y1="-17.78" x2="167.64" y2="-15.24" width="0.1524" layer="91"/>
+<junction x="167.64" y="20.32"/>
+<junction x="167.64" y="17.78"/>
+<junction x="167.64" y="12.7"/>
+<junction x="167.64" y="-12.7"/>
+<junction x="167.64" y="-15.24"/>
 </segment>
 </net>
@@
 <pinref part="IC11" gate="G$1" pin="GND"/>
 <wire x1="172.72" y1="50.8" x2="175.26" y2="50.8" width="0.1524" layer="91"/>
-<wire x1="172.72" y1="50.8" x2="172.72" y2="22.86" width="0.1524" layer="91"/>
+<wire x1="172.72" y1="50.8" x2="172.72" y2="15.24" width="0.1524" layer="91"/>
 <pinref part="IC12" gate="G$1" pin="GND"/>
-<wire x1="172.72" y1="22.86" x2="172.72" y2="20.32" width="0.1524" layer="91"/>
-<wire x1="172.72" y1="20.32" x2="172.72" y2="17.78" width="0.1524" layer="91"/>
-<wire x1="172.72" y1="17.78" x2="172.72" y2="15.24" width="0.1524" layer="91"/>
 <wire x1="172.72" y1="15.24" x2="175.26" y2="15.24" width="0.1524" layer="91"/>
 <wire x1="172.72" y1="15.24" x2="172.72" y2="10.16" width="0.1524" layer="91"/>
@@
 <wire x1="172.72" y1="10.16" x2="172.72" y2="7.62" width="0.1524" layer="91"/>
 <wire x1="172.72" y1="7.62" x2="172.72" y2="5.08" width="0.1524" layer="91"/>
-<wire x1="172.72" y1="5.08" x2="172.72" y2="-12.7" width="0.1524" layer="91"/>
-<wire x1="172.72" y1="-12.7" x2="172.72" y2="-15.24" width="0.1524" layer="91"/>
-<wire x1="172.72" y1="-15.24" x2="172.72" y2="-17.78" width="0.1524" layer="91"/>
-<wire x1="172.72" y1="-17.78" x2="172.72" y2="-20.32" width="0.1524" layer="91"/>
+<wire x1="172.72" y1="5.08" x2="172.72" y2="-20.32" width="0.1524" layer="91"/>
 <wire x1="172.72" y1="-20.32" x2="175.26" y2="-20.32" width="0.1524" layer="91"/>
 <junction x="172.72" y="15.24"/>
-<pinref part="IC12" gate="G$1" pin="I6"/>
-<wire x1="175.26" y1="22.86" x2="172.72" y2="22.86" width="0.1524" layer="91"/>
-<pinref part="IC12" gate="G$1" pin="I7"/>
-<wire x1="175.26" y1="20.32" x2="172.72" y2="20.32" width="0.1524" layer="91"/>
-<pinref part="IC12" gate="G$1" pin="I8"/>
-<wire x1="175.26" y1="17.78" x2="172.72" y2="17.78" width="0.1524" layer="91"/>
-<pinref part="IC13" gate="G$1" pin="I8"/>
-<wire x1="175.26" y1="-17.78" x2="172.72" y2="-17.78" width="0.1524" layer="91"/>
-<pinref part="IC13" gate="G$1" pin="I7"/>
-<wire x1="175.26" y1="-15.24" x2="172.72" y2="-15.24" width="0.1524" layer="91"/>
-<pinref part="IC13" gate="G$1" pin="I6"/>
-<wire x1="175.26" y1="-12.7" x2="172.72" y2="-12.7" width="0.1524" layer="91"/>
-<junction x="172.72" y="-17.78"/>
-<junction x="172.72" y="-15.24"/>
-<junction x="172.72" y="-12.7"/>
-<junction x="172.72" y="17.78"/>
-<junction x="172.72" y="20.32"/>
-<junction x="172.72" y="22.86"/>
 <pinref part="IC9" gate="G$1" pin="GND"/>
 <pinref part="IC8" gate="G$1" pin="GND"/>

Commit message: Attempt to reduce size.
Parts:
- removed R7: 10k, rcl:R-EU_R0805
- removed R8: 4k7, rcl:R-EU_R0805
- added LATCH7, LATCH8, LATCH9: 74HC573D, 74xx-eu:74HC573D
- added R2: 4k7, rcl:R-EU_R0805
- added R3: 10k, rcl:R-EU_R0805
- added SERWIS: 057-010-1, con-panduit:057-010-1
- added ULN7: 1/3, uln-udn2:ULN2803ASOL18
- added ULN8: 2/3, uln-udn2:ULN2803ASOL18
- added ULN9: 3/3, uln-udn2:ULN2803ASOL18
- ULN1: value (none) -> 1/1
- ULN2: value (none) -> 2/1
- ULN3: value (none) -> 3/1
- ULN4: value (none) -> 1/2
- ULN5: value (none) -> 2/2
- ULN6: value (none) -> 3/2
- X1, X2, X3, X4, X5: value 057-010-1 -> 057-016-1; device con-panduit:057-010-1 -> con-panduit:057-016-1; OC_FARNELL unknown -> (none); OC_NEWARK unknown -> (none)
- X6: value 057-010-1 -> 057-016-1; device con-panduit:057-010-1 -> con-panduit:057-016-1
- renumbered IC1 to ATMEGA16, IC10 to ULN3, IC11 to ULN5, IC12 to ULN4, IC13 to ULN6, IC14 to FT232RL, IC2 to LATCH1, IC3 to LATCH3, IC4 to LATCH5, IC5 to LATCH4, IC6 to LATCH2, IC7 to LATCH6, IC8 to ULN2, IC9 to ULN1, X9 to ZASILANIE
Connections:
- removed net N$47 (its old number): ULN4.O3, X3-2.S
- removed net N$61 (its old number): ULN2.O1, X1-2.S
- removed net N$63 (its old number): ULN2.O3, X1-4.S
- removed net N$69 (its old number): ULN2.O4, X1-5.S
- removed net N$70 (its old number): ULN2.O5, X1-6.S
- removed net N$71 (its old number): ULN2.O6, X1-7.S
- removed net N$72 (its old number): ULN2.O7, X1-8.S
- removed net N$73 (its old number): ULN2.O8, X1-9.S
- removed net N$75 (its old number): ULN1.O1, X1-10.S
- removed net N$76 (its old number): ULN1.O2, X2-2.S
- removed net N$77 (its old number): ULN1.O3, X2-3.S
- removed net N$78 (its old number): ULN1.O4, X2-4.S
- removed net N$79 (its old number): ULN1.O5, X2-5.S
- new net N$111: ULN2.O8, X1-6.S
- new net N$112: ULN1.O1, X1-7.S
- new net N$113: ULN1.O2, X1-8.S
- new net N$115: ULN1.O3, X1-10.S
- new net N$116: ULN1.O4, X1-11.S
- new net N$124: LATCH8A.6Q, ULN8.I6
- new net N$128: LATCH8A.7Q, ULN8.I7
- new net N$129: LATCH8A.8Q, ULN8.I8
- new net N$130: LATCH7A.6Q, ULN7.I6
- new net N$131: LATCH7A.7Q, ULN7.I7
- new net N$132: LATCH7A.8Q, ULN7.I8
- new net N$133: ULN1.O5, X1-12.S
- new net N$134: ULN1.O6, X1-14.S
- new net N$135: ULN1.O7, X1-15.S
- new net N$136: ULN1.O8, X1-16.S
- new net N$137: ULN4.O2, X3-3.S
- new net N$138: FT232RL.!RTS
- new net N$139: FT232RL.!CTS
- new net N$140: FT232RL.!DTR
- new net N$141: FT232RL.!DSR
- new net N$142: FT232RL.!DCD
- new net N$143: FT232RL.!RI
- new net N$144: ATMEGA16.(AIN0/INT2)PB2, LATCH7A.6D, LATCH8A.6D, LATCH9A.6D
- new net N$145: ATMEGA16.(T1)PB1, LATCH7A.7D, LATCH8A.7D, LATCH9A.7D
- new net N$146: ATMEGA16.(T0/XCK)PB0, LATCH7A.8D, LATCH8A.8D, LATCH9A.8D
- new net N$147: FT232RL.CBUS0
- new net N$148: FT232RL.CBUS1
- new net N$149: FT232RL.CBUS2
- new net N$150: FT232RL.CBUS3
- new net N$151: FT232RL.CBUS4
- new net N$152: FT232RL.OSCI
- new net N$153: FT232RL.OSCO
- new net N$154: ULN4.O3, X3-4.S
- new net N$155: ULN4.O4, X3-6.S
- new net N$156: ULN4.O5, X3-7.S
- new net N$157: ULN4.O6, X3-8.S
- new net N$158: ULN4.O7, X3-10.S
- new net N$159: ULN4.O8, X3-11.S
- new net N$160: ULN5.O1, X3-12.S
- new net N$161: ULN5.O2, X3-14.S
- new net N$162: ULN5.O3, X3-15.S
- new net N$163: ULN5.O4, X3-16.S
- new net N$164: ULN5.O5, X4-2.S
- new net N$165: ULN5.O6, X4-3.S
- new net N$166: ULN5.O7, X4-4.S
- new net N$167: ULN5.O8, X4-6.S
- new net N$168: ULN6.O1, X4-7.S
- new net N$169: ULN6.O2, X4-8.S
- new net N$170: ULN6.O3, X4-10.S
- new net N$171: ULN6.O4, X4-11.S
- new net N$172: ULN6.O5, X4-12.S
- new net N$173: ULN6.O6, X4-14.S
- new net N$174: ULN6.O7, X4-15.S
- new net N$175: ULN6.O8, X4-16.S
- new net N$176: ULN7.O1, X5-2.S
- new net N$177: ULN7.O2, X5-3.S
- new net N$178: ULN7.O3, X5-4.S
- new net N$179: ULN7.O4, X5-6.S
- new net N$180: ULN7.O5, X5-7.S
- new net N$181: ULN7.O6, X5-8.S
- new net N$182: ULN7.O7, X5-10.S
- new net N$183: ULN7.O8, X5-11.S
- new net N$184: ULN8.O1, X5-12.S
- new net N$185: ULN8.O2, X5-14.S
- new net N$186: ULN8.O3, X5-15.S
- new net N$187: ULN8.O4, X5-16.S
- new net N$188: ULN8.O5, X6-2.S
- new net N$189: ULN8.O6, X6-3.S
- new net N$190: ULN8.O7, X6-4.S
- new net N$191: ULN8.O8, X6-6.S
- new net N$192: ULN9.O1, X6-7.S
- new net N$193: ULN9.O2, X6-8.S
- new net N$194: ULN9.O3, X6-10.S
- new net N$195: ULN9.O4, X6-11.S
- new net N$196: ULN9.O5, X6-12.S
- new net N$197: ULN9.O6, X6-14.S
- new net N$198: ULN9.O7, X6-15.S
- new net N$199: ULN9.O8, X6-16.S
- new net N$53: LATCH4A.6Q, ULN4.I6
- new net N$54: LATCH4A.7Q, ULN4.I7
- new net N$55: LATCH4A.8Q, ULN4.I8
- new net N$56: LATCH8A.1Q, ULN8.I1
- new net N$57: LATCH8A.2Q, ULN8.I2
- new net N$58: LATCH8A.3Q, ULN8.I3
- new net N$59: LATCH8A.4Q, ULN8.I4
- new net N$60: LATCH8A.5Q, ULN8.I5
- new net N$64: LATCH7A.1Q, ULN7.I1
- new net N$65: LATCH7A.2Q, ULN7.I2
- new net N$66: LATCH7A.3Q, ULN7.I3
- new net N$67: LATCH7A.4Q, ULN7.I4
- new net N$68: LATCH7A.5Q, ULN7.I5
- net 12V: now also ULN7.CD+, ULN8.CD+, ULN9.CD+, X1-13.S, X1-5.S, X1-9.S, X2-13.S, X2-5.S, X2-9.S, X3-13.S, X3-5.S, X3-9.S, X4-13.S, X4-5.S, X4-9.S, X5-13.S, X5-5.S, X5-9.S, X6-1.S, X6-13.S, X6-5.S, X6-9.S
- net GND: now also LATCH7A.OC, LATCH8A.OC, LATCH9A.OC, R3.1, SERWIS-10.S, SERWIS-4.S, SERWIS-6.S, SERWIS-8.S, ULN7.GND, ULN8.GND, ULN9.GND; no longer LATCH4A.6D, LATCH4A.7D, LATCH4A.8D, LATCH6A.6D, LATCH6A.7D, LATCH6A.8D, R7.1, X5-10.S, X5-8.S, X5-9.S, X6-10.S, X6-4.S, X6-6.S, X6-8.S
- net N$1: now also LATCH3A.8D
- net N$10: now also LATCH4A.2D, LATCH6A.2D; no longer LATCH3A.2D
- net N$100: now also ULN2.O1, X2-12.S; no longer ULN5.O8, X4-3.S
- net N$101: now also ULN2.O2, X2-14.S; no longer ULN6.O4, X5-6.S
- net N$102: now also ULN2.O3, X2-15.S; no longer ULN4.O1, X2-9.S
- net N$103: now also ULN2.O4, X2-16.S; no longer ULN4.O2, X2-10.S
- net N$104: now also ULN2.O5, X1-2.S; no longer ULN6.O5, X5-7.S
- net N$105: now also SERWIS-7.S; no longer X6-7.S
- net N$106: now also SERWIS-9.S; no longer X6-9.S
- net N$107: now also SERWIS-1.S; no longer X6-1.S
- net N$108: now also ULN2.O6, X1-3.S; no longer ULN6.O1, X5-3.S
- net N$109: now also ULN2.O7, X1-4.S; no longer ULN6.O2, X5-4.S
- net N$11: now also LATCH4A.3D, LATCH6A.3D; no longer LATCH3A.3D
- net N$12: now also LATCH4A.4D, LATCH6A.4D; no longer LATCH3A.4D
- net N$125: now also R2.1, R3.2; no longer R7.2, R8.1
- net N$127: now also SERWIS-5.S; no longer X6-5.S
- net N$13: now also LATCH4A.5D, LATCH6A.5D; no longer LATCH3A.5D
- net N$14: now also LATCH4A.6D, LATCH6A.6D; no longer LATCH3A.6D
- net N$15: now also LATCH4A.7D, LATCH6A.7D; no longer LATCH3A.7D
- net N$16: now also LATCH4A.8D, LATCH6A.8D; no longer LATCH3A.8D
- net N$17: now also LATCH7A.1D, LATCH8A.1D, LATCH9A.1D; no longer LATCH4A.1D, LATCH6A.1D
- net N$18: now also LATCH7A.2D, LATCH8A.2D, LATCH9A.2D; no longer LATCH4A.2D, LATCH6A.2D
- net N$19: now also LATCH7A.3D, LATCH8A.3D, LATCH9A.3D; no longer LATCH4A.3D, LATCH6A.3D
- net N$2: now also LATCH3A.7D
- net N$20: now also LATCH7A.4D, LATCH8A.4D, LATCH9A.4D; no longer LATCH4A.4D, LATCH6A.4D
- net N$21: now also LATCH7A.5D, LATCH8A.5D, LATCH9A.5D; no longer LATCH4A.5D, LATCH6A.5D
- net N$22: now also LATCH5A.C, LATCH8A.C; no longer LATCH3A.C, LATCH4A.C
- net N$23: now also LATCH4A.C, LATCH7A.C; no longer LATCH5A.C, LATCH6A.C
- net N$3: now also LATCH3A.6D
- net N$4: now also LATCH3A.5D
- net N$5: now also LATCH3A.4D
- net N$6: now also LATCH3A.3D
- net N$62: now also ULN4.O1, X3-2.S; no longer ULN2.O2, X1-3.S
- net N$7: now also LATCH3A.2D
- net N$74: now also ATMEGA16.(INT0)PD2, LATCH3A.C, LATCH6A.C, LATCH9A.C; no longer ULN4.O4, X3-3.S
- net N$8: now also LATCH3A.1D
- net N$80: now also LATCH6A.6Q, ULN6.I6; no longer ULN1.O6, X2-6.S
- net N$81: now also LATCH6A.7Q, ULN6.I7; no longer ULN1.O7, X2-7.S
- net N$82: now also LATCH6A.8Q, ULN6.I8; no longer ULN1.O8, X2-8.S
- net N$83: now also ATMEGA16.AREF; no longer ULN4.O5, X3-4.S
- net N$84: now also LATCH9A.1Q, ULN9.I1; no longer ULN3.O1, X4-4.S
- net N$85: now also LATCH9A.2Q, ULN9.I2; no longer ULN3.O2, X4-5.S
- net N$86: now also LATCH9A.3Q, ULN9.I3; no longer ULN3.O3, X4-6.S
- net N$87: now also LATCH9A.4Q, ULN9.I4; no longer ULN3.O4, X4-7.S
- net N$88: now also LATCH9A.5Q, ULN9.I5; no longer ULN3.O5, X4-8.S
- net N$89: now also LATCH9A.6Q, ULN9.I6; no longer ULN3.O6, X4-9.S
- net N$9: now also LATCH4A.1D, LATCH6A.1D; no longer LATCH3A.1D
- net N$90: now also LATCH9A.7Q, ULN9.I7; no longer ULN3.O7, X4-10.S
- net N$91: now also LATCH9A.8Q, ULN9.I8; no longer ULN3.O8, X5-2.S
- net N$92: now also ULN3.O1, X2-2.S; no longer ULN6.O3, X5-5.S
- net N$93: now also ULN3.O2, X2-3.S; no longer ULN5.O1, X3-5.S
- net N$94: now also ULN3.O3, X2-4.S; no longer ULN5.O2, X3-6.S
- net N$95: now also ULN3.O4, X2-6.S; no longer ULN5.O3, X3-7.S
- net N$96: now also ULN3.O5, X2-7.S; no longer ULN5.O4, X3-8.S
- net N$97: now also ULN3.O6, X2-8.S; no longer ULN5.O5, X3-9.S
- net N$98: now also ULN3.O7, X2-10.S; no longer ULN5.O6, X3-10.S
- net N$99: now also ULN3.O8, X2-11.S; no longer ULN5.O7, X4-2.S
- net VCC: now also R2.2, SERWIS-2.S; no longer R8.2, ULN4.I6, ULN4.I7, ULN4.I8, ULN6.I6, ULN6.I7, ULN6.I8, X6-2.S
Other:
- moved on the sheet: C5, C6, L1, X1-1, X1-10, X1-2, X1-3, X1-4, X1-5, X1-6, X1-7, X1-8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
